File: power.kicad_sch (KiCad schematic)
At the start: 21 parts, among them J18 Barrel_Jack_MountingPin, J4 EURO_PWR, U2 AP2204K-3.3, U3 LM1117-5.0, U4 LM4040DBZ-5

Commit message: Gerber files, BOM updated
Added Gerber files, updated the BOM, and fixed the power sheet to have the correct file name.
Parts:
- C10, C14, C4, C8, C9: value 100nF -> (none); footprint Capacitor_SMD:C_0805_2012Metric -> (none)
- C11, C12, C13, C5, C6, C7: value 10uF -> (none); footprint Capacitor_SMD:CP_Elec_5x3 -> (none)
- D1: value MB2S -> (none); footprint Package_TO_SOT_SMD:TO-269AA -> (none)
- J18: value Barrel_Jack_MountingPin -> (none); footprint Connector_BarrelJack:BarrelJack_CLIFF_FC681465S_SMT_Horizontal -> (none)
- J4: value EURO_PWR -> (none); footprint Connector_PinSocket_2.54mm:PinSocket_2x05_P2.54mm_Vertical -> (none)
- L1: value 10uH -> (none); footprint Inductor_SMD:L_0805_2012Metric -> (none)
- PS1: value DLW05A-12 -> (none); footprint DLW05A12 -> (none)
- R6, R7: value 4.7R -> (none); footprint Resistor_SMD:R_0805_2012Metric -> (none)
- U2: value AP2204K-3.3 -> (none); footprint Package_TO_SOT_SMD:SOT-23-5 -> (none)
- U3: value LM1117-5.0 -> (none); footprint Package_TO_SOT_SMD:SOT-223 -> (none)
- U4: value LM4040DBZ-5 -> (none); footprint Package_TO_SOT_SMD:SOT-23 -> (none)

Commit message: various updates
Parts:
- removed U3: (no value), symbol Regulator_Linear:LM1117-5.0
- added U3: LM78L05_SOT, Package_TO_SOT_SMD:SOT-223, symbol Regulator_Linear:LM78L05_TO92
- C10, C14, C4, C8, C9: value (none) -> 100nF; footprint (none) -> Capacitor_SMD:C_0805_2012Metric
- C11, C12, C13, C5, C6, C7: value (none) -> 10uF; footprint (none) -> Capacitor_SMD:CP_Elec_5x3
- D1: value (none) -> MB2S; footprint (none) -> Package_TO_SOT_SMD:TO-269AA
- J18: value (none) -> Barrel_Jack_MountingPin; footprint (none) -> Connector_BarrelJack:BarrelJack_CLIFF_FC681465S_SMT_Horizontal
- J4: value (none) -> EURO_PWR; footprint (none) -> Connector_PinSocket_2.54mm:PinSocket_2x05_P2.54mm_Vertical
- L1: value (none) -> 10uH; footprint (none) -> Inductor_SMD:L_0805_2012Metric
- PS1: value (none) -> DLW05A-12; footprint (none) -> DLW05A12
- R6: value (none) -> 4.7R; footprint (none) -> Resistor_SMD:R_0805_2012Metric
- R7: value (none) -> 2k; footprint (none) -> Resistor_SMD:R_0805_2012Metric
- U2: value (none) -> AP2204K-3.3; footprint (none) -> Package_TO_SOT_SMD:SOT-23-5
- U4: value (none) -> LM4040DBZ-10; footprint (none) -> Package_TO_SOT_SMD:SOT-23
Connections:
- net +5V: now also U3.1 (VO)
- net GNDA: now also U3.2 (GND)
- net at L1.2: now also U3.3 (VI)
